Commit message: l2 lidar: integrate Unitree L2 4D LiDAR into mast + grunt_bringup
URDF: rename lidar_3d_link to l2_mount and reorient for forward-facing
mount on mast front face (cable down). rpy (pi, -pi/2, 0) maps L2 +Z to
robot +X. Driver still publishes its own child l2 frame as identity off
this mount.

Launch + config: prefix-aware grunt_l2.launch.py and grunt_l2_params.yaml
following the gps.rtk pattern. YAML uses /**: wildcard so namespaced node
picks up params. Network is 10.42.0.62/2, IMU publishing enabled,
aggregateNframes=38.

File: grunt_description/urdf/mast.xacro (robot description, xacro)
@@ -91,6 +91,11 @@
     </collision>
   </link>
-  <!-- Unitree L2 4D LiDAR -->
-  <link name="$(arg prefix)lidar_3d_link">
+  <!-- Unitree L2 4D LiDAR — mounting frame.
+       This URDF link carries the L2's physical mounting position + rotation.
+       The driver (markgol's l2lidar_node) publishes one more child below this:
+       $(arg prefix)l2 (the cloud frame), as an identity transform relative
+       to this mount frame. We can't avoid that extra hop without patching the
+       node — its publishStaticTransform() always emits robot_id → frame_id. -->
+  <link name="$(arg prefix)l2_mount">
     <inertial>
       <mass value="0.195"/>
@@ -128,11 +133,21 @@
     <child link="$(arg prefix)imu_link"/>
   </joint>
-  <!-- Unitree L2 LiDAR: on shelf angled 20deg forward-down,
-       4cm forward (+X) of mast center, 34cm above mast base.
-       Pitch = -0.3491 rad tilts front of LiDAR downward. -->
-  <joint name="$(arg prefix)lidar_3d_joint" type="fixed">
-    <origin xyz="0.04 0 0.34" rpy="0 -0.3491 0"/>
+  <!-- Unitree L2 LiDAR: mounted forward-facing on the mast's front
+       vertical face. Mast trapezoid is 50mm deep, so front face is at
+       +X = 0.025m in mast base_link. L2 base center on that face at
+       Y = 0, Z = 0.34m above mast base. Cable points straight down.
+       Rotation rpy=(pi, -pi/2, 0) maps the L2's coordinate system into
+       the robot frame:
+         L2 +Z (out of mounting surface) → robot +X (forward)
+         L2 +X (opposite the cable exit) → robot +Z (up, since cable is down)
+         L2 +Y                            → robot -Y
+       So the L2's hemispherical FOV is centered on robot +X (forward-looking).
+       Note: there's a ~few-degree CCW (viewed from behind) yaw error from
+       hand-drilled mounting holes; will be eliminated by a CNC'd plate.
+       Ignored here. -->
+  <joint name="$(arg prefix)l2_mount_joint" type="fixed">
+    <origin xyz="0.025 0 0.34" rpy="${pi} ${-pi/2} 0"/>
     <parent link="$(arg prefix)base_link"/>
-    <child link="$(arg prefix)lidar_3d_link"/>
+    <child link="$(arg prefix)l2_mount"/>
   </joint>
 </robot>

Commit message: grunt_l2: migrate to V0.5 single-frame geometry
l2lidar_node V0.5 collapses its parameter surface to l2_name /
cloud_frame / publish_tf and emits only the intrinsic cloud→imu static
TF — URDF now owns the extrinsic placement. This commit threads the
Grunt-side wiring through that change.

mast.xacro: rename URDF link l2_mount → l2 (matching joint l2_joint).
The mount + the cloud frame are now the same link (Unitree spec; no
mount-to-cloud offset). Note: we deliberately keep `l2` as the local
name rather than adopt the upstream V0.5 default `l2lidar_link`, so
existing bags, rviz/Foxglove layouts, and Nav2 layer configs keep
working without a sweep. The IMU frame auto-derives to `l2_imu`
(no `_link` suffix to strip → driver just appends `_imu`).

grunt_l2.launch.py: replace the V0.3.x param dict — robot_id/frame_id/
imu_frame_id/robot_x/y/z — with the V0.5 surface (cloud_frame +
publish_tf). cloud_frame is set to [prefix, "/mast/l2"] for the
existing Grunt frame-naming convention.

Net TF chain (down from 3 hops to 2):
  <prefix>/mast/base_link
    → <prefix>/mast/l2          (URDF — also the cloud frame)
    → <prefix>/mast/l2_imu      (driver — intrinsic L2 IMU offset)

File: grunt_description/urdf/mast.xacro (robot description, xacro)
@@ -91,11 +91,15 @@
     </collision>
   </link>
-  <!-- Unitree L2 4D LiDAR — mounting frame.
-       This URDF link carries the L2's physical mounting position + rotation.
-       The driver (markgol's l2lidar_node) publishes one more child below this:
-       $(arg prefix)l2 (the cloud frame), as an identity transform relative
-       to this mount frame. We can't avoid that extra hop without patching the
-       node — its publishStaticTransform() always emits robot_id → frame_id. -->
-  <link name="$(arg prefix)l2_mount">
+  <!-- Unitree L2 4D LiDAR — primary reference frame.
+       Per Unitree's spec, the L2's point-cloud coordinate origin is the
+       geometric center of its bottom mounting surface, so this URDF link
+       is both the mounting reference AND the cloud frame. Under V0.5 of
+       markgol's l2lidar_node, the driver publishes only one child below
+       this link (the IMU frame, at the documented intrinsic offset); the
+       old `l2_mount → l2` identity-TF workaround is gone.
+       Frame name is `l2` (not the upstream-default `l2lidar_link`) for
+       downstream-consumer continuity — existing bags, rviz/Foxglove
+       layouts, and Nav2 layer configs all reference `<prefix>/mast/l2`. -->
+  <link name="$(arg prefix)l2">
     <inertial>
       <mass value="0.195"/>
@@ -146,8 +150,8 @@
        hand-drilled mounting holes; will be eliminated by a CNC'd plate.
        Ignored here. -->
-  <joint name="$(arg prefix)l2_mount_joint" type="fixed">
+  <joint name="$(arg prefix)l2_joint" type="fixed">
     <origin xyz="0.025 0 0.34" rpy="${pi} ${-pi/2} 0"/>
     <parent link="$(arg prefix)base_link"/>
-    <child link="$(arg prefix)l2_mount"/>
+    <child link="$(arg prefix)l2"/>
   </joint>
 </robot>

Commit message: grunt_description: point L2 mesh at l2lidar_node's installed STL
Drop grunt_description's local copy of unitreeL2.stl (1.28 MB, pre-V0.5
mesh) in favor of l2lidar_node's canonical mesh at
package://l2lidar_node/meshes/l2_lidar.stl (486 KB, Medium-refinement
Fusion 360 export, origin at bottom mounting surface = cloud-frame
origin). Shipped upstream via PR #8.

Single source of truth — future upstream mesh updates land in Grunt
automatically. Add l2lidar_node as exec_depend so the share dir is
guaranteed present at runtime.

File: grunt_description/urdf/mast.xacro (robot description, xacro)
@@ -112,5 +112,5 @@
       <origin xyz="0 0 0" rpy="0 0 0"/>
       <geometry>
-        <mesh filename="package://grunt_description/meshes/unitreeL2.stl"/>
+        <mesh filename="package://l2lidar_node/meshes/l2_lidar.stl"/>
       </geometry>
       <material name="$(arg prefix)black"/>
